File: PCB_project/PTR_nano.kicad_pcb (KiCad board)
At the start: 6 copper layers, 16 x 11 mm, 65 parts, among them J1 ESP32_PROG_CON, J2 BAT, J3 IGN, J4 IGN, Q1 CSD13380F3, Q2 CSD13380F3, Q3 CSD13380F3, Q4 CSD13380F3, U1 ESP8685H4, U2 LSM6DSO32, U3 BMP280, U4 NCP161AMX330TBG, Y1 XRCGB40M000F4M00R0

Commit message: Board name fix
Other:
- board text added: "nano"
- board text removed: "mini"
Changed lines of the file:
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@@
 		)
 	)
-	(gr_text "mini"
+	(gr_text "nano"
 		(at 136 89.25 90)
 		(layer "B.SilkS")
