File: PTR_nano_pcb/PTR_nano_pcb.kicad_pcb (KiCad board)
At the start: 6 copper layers, 16 x 11 mm, 65 parts, among them J1 ESP32_PROG_CON, J2 BAT, J3 IGN, J4 IGN, Q1 CSD13380F3, Q2 CSD13380F3, Q3 CSD13380F3, Q4 CSD13380F3, U1 ESP8685H4, U2 LSM6DSO32, U3 BMP280, U4 NCP161AMX330TBG, Y1 XRCGB40M000F4M00R0

Commit message: Pressure sensor changed to BMP581
+ library fixed
Parts:
- removed U3: BMP280, Package_LGA:Bosch_LGA-8_2x2.5mm_P0.65mm_ClockwisePinNumbering
- added U5: BMP581, PTR_nano_footprint:BMP581, F.Cu at (142.9, 94.7)
Routing:
- net SPI_CS_BMP: track 4.22 -> 8.59 mm, vias 0 -> 2
- net GND: track 15.4 -> 13.6 mm, vias 26 -> 24
- net SPI_MISO: track 7.20 -> 6.40 mm
- net SPI_CLK: track 5.68 -> 6.44 mm
- removed copper zone on F.Cu, net +3V3
- removed copper zone on B.Cu, net +BATT
- removed copper zone on In1.Cu, net +BATT
- removed copper zone on In2.Cu, net +BATT
- removed copper zone on In2.Cu, net GND
- removed copper zone on F.Cu, net VBAT
